File: pi_power_hat.kicad_pcb (KiCad board)
At the start: 2 copper layers, 92.5 x 30 mm, 24 parts, among them J1 GPIO_CONNECTOR, J2 Barrel_Jack, J3 PIR Motion Sensor, J4 DH22T, J5 Screw_Terminal_01x02, Q1 DMG1012UW-7

Commit message: Update
Other:
- net class Default removed
